File: pcb/pcb.kicad_sch (KiCad schematic)
At the start: 121 parts

Commit message: updated bom, plate
Parts:
- C0, C1: value (none) -> 22pf; footprint (none) -> Capacitor_SMD:C_0805_2012Metric
- C2: value (none) -> 1uf; footprint (none) -> Capacitor_SMD:C_0805_2012Metric
- C3, C4: value (none) -> .1uf / 100nf; footprint (none) -> Capacitor_SMD:C_0805_2012Metric
- C5: value (none) -> 10uf; footprint (none) -> Capacitor_SMD:C_0805_2012Metric
- D1, D10011, D1011, D110111, D112113, D114, D12013, D1213, D14, D1415, D1617, D1819, D2021, D203, D211212, D213214, D2324, D2526, D2728, D29210, D3031, D311312, D313314, D3334, D3536, D3738, D39310, D4041, D405, D410411, D412413, D414, D4344, D607, D809: value (none) -> BAV70_Small; footprint (none) -> Package_TO_SOT_SMD:SOT-23
- F0: value (none) -> Polyfuse; footprint (none) -> Fuse:Fuse_1206_3216Metric
- J0: value (none) -> USB_C_Receptacle_USB2.0; footprint (none) -> Connector_USB:USB_C_Receptacle_HRO_TYPE-C-31-M-12
- K0,0, K0,1, K0,10, K0,11, K0,12, K0,13, K0,14, K0,2, K0,3, K0,4, K0,5, K0,6, K0,7, K0,8, K0,9, K1,0, K1,1, K1,10, K1,11, K1,12, K1,13, K1,14, K1,2, K1,3, K1,4, K1,5, K1,6, K1,7, K1,8, K1,9, K2,0, K2,10, K2,11, K2,12, K2,13, K2,14, K2,2, K2,3, K2,4, K2,5, K2,6, K2,7, K2,8, K2,9, K3,0, K3,10, K3,11, K3,12, K3,13, K3,14, K3,2, K3,3, K3,4, K3,5, K3,6, K3,7, K3,8, K3,9, K4,0, K4,10, K4,11, K4,12, K4,13, K4,14, K4,2, K4,3, K4,4: value (none) -> KEYSW; footprint (none) -> kbd:keyswitch_cherrymx_alps_combo_fixed
- R0, R5: value (none) -> 10k; footprint (none) -> Resistor_SMD:R_0805_2012Metric
- R1, R2: value (none) -> 22; footprint (none) -> Resistor_SMD:R_0805_2012Metric
- R3, R4: value (none) -> 5.1k; footprint (none) -> Resistor_SMD:R_0805_2012Metric
- SW0: value (none) -> SW_PUSH; footprint (none) -> Keebio-Parts:SW_SPST_TL3342
- U0: value (none) -> ATmega32U2-A; footprint (none) -> Package_QFP:TQFP-32_7x7mm_P0.8mm
- U1: value (none) -> SRV05-4; footprint (none) -> Package_TO_SOT_SMD:SOT-23-6
- Y0: value (none) -> Crystal_GND24_Small; footprint (none) -> Crystal:Crystal_SMD_3225-4Pin_3.2x2.5mm
- j1: LCSC C160404 -> C2845363
