File: pcb/plate.kicad_pcb (KiCad board)
At the start: 2 copper layers, 304.8 x 95.2 mm, 8 parts

Commit message: updated bom, plate
Routing:
- added copper zone on B.Cu, net GND
- added copper zone on F.Cu, net GND
Changed lines of the file:
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@@
   (gr_line (start 54.6625 54.025) (end 69.1625 54.025) (layer "Edge.Cuts") (width 0.2))
   (gr_arc (start 17.275 15.425) (mid 17.128553 15.778553) (end 16.775 15.925) (layer "Edge.Cuts") (width 0.2))
+  (zone (net 1) (net_name "GND") (layers F&B.Cu) (hatch edge 0.508)
+    (connect_pads (clearance 0.508))
+    (min_thickness 0.254) (filled_areas_thickness no)
+    (fill yes (mode hatch) (thermal_gap 0.508) (thermal_bridge_width 0.508)
+      (hatch_thickness 1.016) (hatch_gap 1.524) (hatch_orientation 45)
+      (hatch_border_algorithm hatch_thickness) (hatch_min_hole_area 0.3))
+    (polygon
+      (pts
+        (xy 316.9 121)
+        (xy -21 121)
+        (xy -21 -15.3)
+        (xy 316.9 -15.3)
+      )
+    )
+  )
 )
